Commit message: Actividad 10: Integración definitiva de COLMIBOT en Gazebo Harmonic con físicas y colisiones corregidas.

File: robot_description/robot_description/urdf/colmibot.urdf (robot description, URDF)
Before this commit: robot colmibot, 8 links, 7 joints
Links:
- link base_link: mass None -> 0.084; geometry collision box size=0.2 0.15 0.1; visual mesh filename=package://robot_description/meshes/CLM-Body.stl name=body_mesh scale=0.001 0.001 0.001
- link camera_link: mass None -> 0.1814
- link holder_link: mass None -> 0.0136
- link plato_inferior_link: mass None -> 0.0821
- link plato_superior_link: mass None -> 0.0821
- link wheel_left_link: mass None -> 0.0195; geometry collision cylinder length=0.02 radius=0.03; visual mesh filename=package://robot_description/meshes/CLM-Llanta60mmD.stl name=wheel_l_mesh scale=0.001 0.001 0.001
- link wheel_right_link: mass None -> 0.0195; geometry collision cylinder length=0.02 radius=0.03; visual mesh filename=package://robot_description/meshes/CLM-Llanta60mmD.stl name=wheel_r_mesh scale=0.001 0.001 0.001
Joints:
- joint wheel_left_joint: origin xyz=0.0 0.078 0.015 rpy=0 0 0 -> xyz=0 0.11 0 rpy=0 0 0
- joint wheel_right_joint: origin xyz=0.0 -0.078 0.015 rpy=0 0 0 -> xyz=0 -0.11 0 rpy=0 0 0
